File: ptFlex/ptFlex.kicad_sch (KiCad schematic)
At the start: 72 parts, among them J1 Barrel_Jack_Switch, J2 Programming, J3 Qwiic, J4 6 Pin Male Header, Q1 MMBT3904, Q2 MMBT3904, Q3 DMP2004K-7, Q4 BSS138, Q5 BSS138, U1 LM1086-5.0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

Commit message: Updating to PCB 2.0.1 to fix missing I2C wires.
Parts:
- U1: LCSC C5145331 -> C434504
Changed lines of the file:
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@@
 			)
 		)
-		(property "LCSC" "C5145331"
+		(property "LCSC" "C434504"
 			(at 220.98 184.15 0)
 			(effects

Commit message: Finalizing PCB v2.0.2. Including some minor tweaks to the firmware as well.
Parts:
- added C26: 1uF, Capacitor_SMD:C_0805_2012Metric, symbol Device:C
- added J5: Rx Aud, Connector_PinHeader_2.54mm:PinHeader_1x02_P2.54mm_Vertical, symbol Connector_Generic:Conn_01x02
- added R22, R23: 10k, Resistor_SMD:R_0805_2012Metric, symbol Device:R_US
Connections:
- net +5V: now also R22.2
- net GND: now also J5.2 (Pin_2), R23.1
- net XMIT-RX-AUDIO: now reaches U3.23 (PC0)
- net XMIT-RX-AUDIO: now also C26.1, R22.1, R23.2
- net at U5.3 (AF-OUT): now also C26.2, J5.1 (Pin_1)
Other:
- moved on the sheet: C18, Q2, R14, R15

Commit message: Updated BOM parts
Parts:
- U1: LCSC C434504 -> C22446570
Changed lines of the file:
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@@
 			)
 		)
-		(property "LCSC" "C434504"
+		(property "LCSC" "C22446570"
 			(at 220.98 184.15 0)
 			(effects
